File: const-led-ez/const-led.sch (KiCad schematic (older format))
At the start: 25 parts, among them CON1 AVR-ISP-6, J1 Micro_USB_B, J2 Conn_01x02, SW1 SW_SPST, SW2 SW_SPST, U1 MCP73831, U2 LM3410, U3 ATTINY85-20SU

Commit message: Rev2
Parts:
- removed D1: D_Schottky, Diodes_SMD:D_SMA, symbol D_Schottky
- added D6: LED, personal_f:ChanzonLED, symbol LED
- added J3: Conn_01x02, Pin_Headers:Pin_Header_Straight_1x02_Pitch2.54mm, symbol Conn_01x02
- added J4, J5, J6, J7: Conn_01x01, Mounting_Holes:MountingHole_3.2mm_M3, symbol Conn_01x01
- added J8, J9: Conn_01x01, personal_f:VIA-12mil, symbol Conn_01x01
- added Q1: QS5U28, TO_SOT_Packages_SMD:TSOT-23-5, symbol QS5U28
- added R5: 100k, Resistors_SMD:R_0603, symbol R
- D3: value D_Schottky -> 1N5819; footprint Diodes_SMD:D_SMA -> Diodes_SMD:D_SOD-123
- D4: footprint Pin_Headers:Pin_Header_Straight_1x02_Pitch2.54mm -> personal_f:ChanzonLED
- L1: value 16u -> 4u; footprint personal_f:muRata_L -> Inductors_SMD:L_0805
- R9: value R -> 1k
- SW1: footprint Pin_Headers:Pin_Header_Straight_1x02_Pitch2.54mm_SMD_Pin1Left -> Buttons_Switches_SMD:SW_SPDT_PCM12
- SW2: footprint Pin_Headers:Pin_Header_Straight_1x02_Pitch2.54mm_SMD_Pin1Left -> Buttons_Switches_SMD:SW_SPST_B3S-1000
Connections:
- net FB: now also D6.1 (K), J3.1 (Pin_1); no longer D4.1 (K)
- net GND: now also R5.2
- net MISO: now also TP1.1
- net VBAT: now also Q1.5 (D); no longer SW1.1 (A)
- net VCC: no longer CON1.2
- net at C4.1, D3.1 (K), D4.2 (A): now also J3.2 (Pin_2)
- net V_USB: now reaches J1.1 (VBUS)
- net V_USB: now also C1.1, CON1.2, D2.2 (A), U1.4 (VDD), Q1.1 (G), Q1.3, R5.1
- removed net VIN: C1.1, D2.2 (A), TP1.1, U1.4 (VDD)
- new net: D4.1 (K), D6.2 (A)
- new net: Q1.2 (S), Q1.4, SW1.1 (A)
- new net THERM: J8.1 (Pin_1), J9.1 (Pin_1)
- no-connect marks 0 -> 3
Other:
- note added: "Power OR"
- note added: "Use 1.6 MHz version."
- moved on the sheet: C1, C2, C4, D2, J1, J2, R1, R2, SW1, U1
